File: pcb.kicad_pcb (KiCad board)
At the start: 2 copper layers, 22.4 x 43 mm, 13 parts, among them J1 vik-module-connector, J2 Conn_01x12_Pin, J3 vik-module-connector, Q1 S8050

Commit message: v0.2
Parts:
- removed R2: 1k, Resistor_SMD:R_1206_3216Metric_Pad1.30x1.75mm_HandSolder
- removed R3: 10k, Resistor_SMD:R_1206_3216Metric_Pad1.30x1.75mm_HandSolder
- moved R1 4.00 mm to (105.5, 63.0), turned to -90 degrees
- moved Q1 3.42 mm to (99.5, 61.6)
- moved JP1 3.00 mm to (99.5, 56.8), turned to 180 degrees
- moved C2 0.20 mm to (107.5, 82.6)
Connections:
- JP1 pad 1: Net-(JP1-A) -> GND
- JP1 pad 2: GND -> Net-(JP1-B)
- Q1 pad 2: Net-(Q1-B) -> BLK
- Q1 pad 3: Net-(JP1-A) -> Net-(JP1-B)
- R1 pad 1: Net-(JP1-A) -> Net-(JP1-B)
Routing:
- net +3.3V: track 57.2 -> 40.4 mm
- net Net-(JP1-B): track 0.00 -> 11.7 mm
- net Net-(JP1-A): track 9.77 -> 0.00 mm
- net Net-(Q1-B): track 8.87 -> 0.00 mm
- net LEDK: track 31.4 -> 27.7 mm
- net DC: track 28.4 -> 25.7 mm
- net MOSI: track 21.7 -> 20.6 mm
- net BLK: track 16.2 -> 15.2 mm
Other:
- board text added: "v0.2"
