File: pcb/1.47inch/pcb.kicad_pcb (KiCad board)
At the start: 2 copper layers, 22 x 39 mm, 17 parts, among them J1 vik-module-connector, J2 vik-module-connector, J3 Conn_01x12_Pin, Q1 S8050

Commit message: small updates
Parts:
- moved TP5 0.20 mm to (95.7, 62.2)
Other:
- board text added: "v1.1"
- board text removed: "v1.0"
Changed lines of the file:
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@@
         (effects (font (size 1 1) (thickness 0.15)) (justify mirror))
     )
-    (pad "" thru_hole circle (at 0 0 180) (size 4.5 4.5) (drill 2.6) (layers "*.Cu" "B.Mask"))
+    (pad "" thru_hole circle (at 0 0 180) (size 4.8 4.8) (drill 2.65) (layers "*.Cu" "B.Mask"))
     (model "${ZZKEEB}/models/solder-nut-4x5x2.5x1.5.step"
       (offset (xyz 0 0 0))
@@
   )
   (footprint "TestPoint:TestPoint_Pad_D1.5mm" (layer "B.Cu")
-    (at 95.5 62.2 180)
+    (at 95.7 62.2 180)
     (descr "SMD pad as test Point, diameter 1.5mm")
     (tags "test point SMD pad")
@@
         (effects (font (size 1 1) (thickness 0.15)) (justify mirror))
     )
-    (pad "" thru_hole circle (at 0 0 180) (size 4.5 4.5) (drill 2.6) (layers "*.Cu" "B.Mask"))
+    (pad "" thru_hole circle (at 0 0 180) (size 4.8 4.8) (drill 2.65) (layers "*.Cu" "B.Mask"))
     (model "${ZZKEEB}/models/solder-nut-4x5x2.5x1.5.step"
       (offset (xyz 0 0 0))
@@
     )
   )
+  (gr_circle (center 109.7 67.4) (end 110.2 67.4)
+    (stroke (width 0.15) (type default)) (fill none) (layer "B.SilkS"))
+  (gr_circle (center 109.7 69.8) (end 110.2 69.8)
+    (stroke (width 0.15) (type default)) (fill none) (layer "B.SilkS"))
+  (gr_arc (start 109.040404 69.6) (mid 108.700449 68.521023) (end 108.990253 67.427509)
+    (stroke (width 0.15) (type default)) (layer "B.SilkS"))
   (gr_line (start 89.5 95.2) (end 91 95.2)
     (stroke (width 0.1) (type default)) (layer "Edge.Cuts"))
@@
   (gr_rect (start 89.8 57.2) (end 109.2 93.5)
     (stroke (width 0.05) (type default)) (fill none) (layer "F.CrtYd"))
-  (gr_text "v1.0" (at 108.9 91.2 90) (layer "B.SilkS")
+  (gr_text "v1.1" (at 108.9 91.2 90) (layer "B.SilkS")
     (effects (font (size 1.5 1.5) (thickness 0.3) bold) (justify mirror))
   )
@@
   (segment (start 97.7 80.8) (end 98.25 80.25) (width 0.2) (layer "B.Cu") (net 10))
   (segment (start 98.25 69.4) (end 98.25 61.4) (width 0.2) (layer "B.Cu") (net 10))
+  (segment (start 96.5 62.2) (end 97.55 61.15) (width 0.2) (layer "B.Cu") (net 10))
   (segment (start 98.25 80.25) (end 98.25 79.6) (width 0.2) (layer "B.Cu") (net 10))
+  (segment (start 97.55 61.15) (end 98.5 61.15) (width 0.2) (layer "B.Cu") (net 10))
   (segment (start 95.5 62.2) (end 96.5 62.2) (width 0.2) (layer "B.Cu") (net 10))
-  (segment (start 97.55 61.15) (end 98.5 61.15) (width 0.2) (layer "B.Cu") (net 10))
-  (segment (start 96.5 62.2) (end 97.55 61.15) (width 0.2) (layer "B.Cu") (net 10))
   (segment (start 98.25 61.4) (end 98.5 61.15) (width 0.2) (layer "B.Cu") (net 10))
   (segment (start 98.25 71.738) (end 98.25 69.4) (width 0.2) (layer "B.Cu") (net 10))
