File: pcb/2inch-0.8mm/pcb.kicad_pcb (KiCad board)
At the start: 2 copper layers, 22 x 33 mm, 17 parts, among them J1 vik-module-connector, J2 vik-module-connector, J3 Conn_01x12_Pin, Q1 S8050

Commit message: small updates
Parts:
- moved C1 0.60 mm to (91.5, 67.2)
- moved TP5 0.20 mm to (95.7, 64.2)
Routing:
- net BLK: track 27.0 -> 26.3 mm
- net RESET: track 20.7 -> 20.1 mm
Changed lines of the file:
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@@
         (effects (font (size 1 1) (thickness 0.15)) (justify mirror))
     )
-    (pad "" thru_hole circle (at 0 0 180) (size 4.5 4.5) (drill 2.6) (layers "*.Cu" "B.Mask"))
+    (pad "" thru_hole circle (at 0 0 180) (size 4.8 4.8) (drill 2.65) (layers "*.Cu" "B.Mask"))
     (model "${ZZKEEB}/models/solder-nut-4x5x2.5x1.5.step"
       (offset (xyz 0 0 0))
@@
   )
   (footprint "TestPoint:TestPoint_Pad_D1.5mm" (layer "B.Cu")
-    (at 95.5 64.2 180)
+    (at 95.7 64.2 180)
     (descr "SMD pad as test Point, diameter 1.5mm")
     (tags "test point SMD pad")
@@
   )
   (footprint "Capacitor_SMD:C_1206_3216Metric_Pad1.33x1.80mm_HandSolder" (layer "B.Cu")
-    (at 91.5 66.6 -90)
+    (at 91.5 67.2 -90)
     (descr "Capacitor SMD 1206 (3216 Metric), square (rectangular) end terminal, IPC_7351 nominal with elongated pad for handsoldering. (Body size source: IPC-SM-782 page 76, https://www.pcb-3d.com/wordpress/wp-content/uploads/ipc-sm-782a_amendment_1_and_2.pdf), generated with kicad-footprint-generator")
     (tags "capacitor handsolder")
@@
         (effects (font (size 1 1) (thickness 0.15)) (justify mirror))
     )
-    (pad "" thru_hole circle (at 0 0 180) (size 4.5 4.5) (drill 2.6) (layers "*.Cu" "B.Mask"))
+    (pad "" thru_hole circle (at 0 0 180) (size 4.8 4.8) (drill 2.65) (layers "*.Cu" "B.Mask"))
     (model "${ZZKEEB}/models/solder-nut-4x5x2.5x1.5.step"
       (offset (xyz 0 0 0))
@@
     )
   )
+  (gr_circle (center 109.5 71.8) (end 110 71.8)
+    (stroke (width 0.15) (type default)) (fill none) (layer "B.SilkS"))
+  (gr_circle (center 109.5 69.4) (end 110 69.4)
+    (stroke (width 0.15) (type default)) (fill none) (layer "B.SilkS"))
+  (gr_arc (start 108.840404 71.6) (mid 108.500427 70.521024) (end 108.790253 69.427509)
+    (stroke (width 0.15) (type default)) (layer "B.SilkS"))
   (gr_line (start 109.5 58.2) (end 89.5 58.2)
     (stroke (width 0.1) (type default)) (layer "Edge.Cuts"))
@@
     (effects (font (size 1 1) (thickness 0.15) bold))
   )
-  (segment (start 92.55 71.65) (end 91.5 71.65) (width 0.2) (layer "B.Cu") (net 1))
   (segment (start 97.9 84.2) (end 92.9 79.2) (width 0.2) (layer "B.Cu") (net 1))
+  (segment (start 92.9 72) (end 92.55 71.65) (width 0.2) (layer "B.Cu") (net 1))
+  (segment (start 91.5 71.65) (end 91.5 68.7625) (width 0.2) (layer "B.Cu") (net 1))
   (segment (start 97.9 85.6) (end 97.9 84.2) (width 0.2) (layer "B.Cu") (net 1))
   (segment (start 92.9 79.2) (end 92.9 72) (width 0.2) (layer "B.Cu") (net 1))
-  (segment (start 92.9 72) (end 92.55 71.65) (width 0.2) (layer "B.Cu") (net 1))
-  (segment (start 91.5 71.65) (end 91.5 68.1625) (width 0.2) (layer "B.Cu") (net 1))
+  (segment (start 92.55 71.65) (end 91.5 71.65) (width 0.2) (layer "B.Cu") (net 1))
   (segment (start 101.85 85.6) (end 101.85 88) (width 0.2) (layer "B.Cu") (net 2))
   (segment (start 101.5 71) (end 101.75 71.25) (width 0.2) (layer "B.Cu") (net 2))
@@
   (via (at 98.25 69.4) (size 0.8) (drill 0.4) (layers "F.Cu" "B.Cu") (net 10))
   (via (at 98.1 80.8) (size 0.8) (drill 0.4) (layers "F.Cu" "B.Cu") (net 10))
+  (segment (start 95.7 64.2) (end 95.7 64) (width 0.2) (layer "B.Cu") (net 10))
+  (segment (start 97.55 62.15) (end 98.5 62.15) (width 0.2) (layer "B.Cu") (net 10))
   (segment (start 98.25 62.4) (end 98.25 69.4) (width 0.2) (layer "B.Cu") (net 10))
   (segment (start 98.25 80.65) (end 98.25 79.6) (width 0.2) (layer "B.Cu") (net 10))
   (segment (start 98.1 80.8) (end 98.25 80.65) (width 0.2) (layer "B.Cu") (net 10))
-  (segment (start 95.5 64.2) (end 95.5 63.2) (width 0.2) (layer "B.Cu") (net 10))
-  (segment (start 95.5 63.2) (end 96.55 62.15) (width 0.2) (layer "B.Cu") (net 10))
+  (segment (start 95.7 64) (end 97.55 62.15) (width 0.2) (layer "B.Cu") (net 10))
   (segment (start 98.5 62.15) (end 98.25 62.4) (width 0.2) (layer "B.Cu") (net 10))
-  (segment (start 96.55 62.15) (end 98.5 62.15) (width 0.2) (layer "B.Cu") (net 10))
   (segment (start 98.25 71.738) (end 98.25 69.4) (width 0.2) (layer "B.Cu") (net 10))
-  (segment (start 107.5 66.15) (end 106.45 66.15) (width 0.2) (layer "B.Cu") (net 20))
-  (segment (start 106.45 66.15) (end 101.5 61.2) (width 0.2) (layer "B.Cu") (net 20))
-  (segment (start 101.5 61.2) (end 100.5 61.2) (width 0.2) (layer "B.Cu") (net 20))
+  (segment (start 104.95 66.15) (end 100.5 61.7) (width 0.2) (layer "B.Cu") (net 20))
+  (segment (start 100.5 61.7) (end 100.5 61.2) (width 0.2) (layer "B.Cu") (net 20))
+  (segment (start 107.5 66.15) (end 104.95 66.15) (width 0.2) (layer "B.Cu") (net 20))
   (zone (net 2) (net_name "GND") (layer "B.Cu") (hatch edge 0.5)
     (connect_pads (clearance 0.5))
